Commit message: Backup phase-one SLAM and navigation experiments

File: src/lunar_rover_description/urdf/lunar_rover.urdf.xacro (robot description, xacro)
@@ -294,5 +294,5 @@
     <parent link="sensor_mast_link"/>
     <child link="mid360_link"/>
-    <origin xyz="0 0 0.155" rpy="0 ${pi / 4.0} 0"/>
+    <origin xyz="0 0 0.155" rpy="0 ${35.0 * pi / 180.0} 0"/>
   </joint>
   <link name="livox_frame"/>

Commit message: chore: backup calibrated odometry and direct teleop

File: src/lunar_rover_description/urdf/lunar_rover.urdf.xacro (robot description, xacro)
@@ -13,5 +13,5 @@
   <xacro:property name="middle_x" value="0.00"/>
   <xacro:property name="rocker_y" value="0.135"/>
-  <xacro:property name="wheel_radius" value="0.075"/>
+  <xacro:property name="wheel_radius" value="0.0625"/>
   <xacro:property name="wheel_width" value="0.055"/>
   <xacro:property name="wheel_mass" value="0.70"/>
