Commit message: feat: add multi-sensor cloud fusion, elevation grid, and image cave ceiling
- Add multisensor_cloud_fusion_node (LiDAR-constrained camera depth fusion)
  with config and unit tests (enable_cloud_fusion defaults to false)
- Extend elevation_grid_node (C++) and terrain_mapper_node with slope/roughness
- Add image_cave lidar ceiling model (STL/DAE meshes)
- Update bringup/restart scripts, launch files, and docs

File: src/lunar_rover_description/Rover_0/urdf/lunar_rover.urdf.xacro (robot description, xacro)
@@ -311,5 +311,6 @@
     <visual>
       <geometry>
-        <box size="0.035 0.12 0.032"/>
+        <!-- Gemini 335: D x W x H = 30 x 90 x 25 mm. -->
+        <box size="0.030 0.090 0.025"/>
       </geometry>
       <material name="camera_black"/>
@@ -317,8 +318,8 @@
     <collision>
       <geometry>
-        <box size="0.035 0.12 0.032"/>
+        <box size="0.030 0.090 0.025"/>
       </geometry>
     </collision>
-    <xacro:box_inertial mass="0.30" x="0.035" y="0.12" z="0.032"/>
+    <xacro:box_inertial mass="0.097" x="0.030" y="0.090" z="0.025"/>
   </link>
   <joint name="gemini335_joint" type="fixed">
@@ -331,5 +332,5 @@
     <parent link="gemini335_link"/>
     <child link="gemini335_color_optical_frame"/>
-    <origin xyz="0.0175 0 0" rpy="${-pi / 2.0} 0 ${-pi / 2.0}"/>
+    <origin xyz="0.015 0 0" rpy="${-pi / 2.0} 0 ${-pi / 2.0}"/>
   </joint>
   <link name="gemini335_depth_optical_frame"/>
@@ -630,4 +631,5 @@
         <camera>
           <optical_frame_id>gemini335_color_optical_frame</optical_frame_id>
+          <!-- Depth-priority profile: Gemini 335 640x400 is a 90 x 65 deg mode. -->
           <horizontal_fov>${90.0 * pi / 180.0}</horizontal_fov>
           <image>
@@ -637,6 +639,7 @@
           </image>
           <clip>
-            <near>0.10</near>
-            <far>10.0</far>
+            <!-- Official Minimum-Z for 640x400 is 0.26 m; nominal range reaches 20 m+. -->
+            <near>0.26</near>
+            <far>20.0</far>
           </clip>
           <noise>
@@ -644,5 +647,6 @@
             <mean>0.0</mean>
             <xacro:if value="$(arg sensor_noise)">
-              <stddev>0.003</stddev>
+              <!-- Conservative 1.5% spatial precision bound at 2 m. -->
+              <stddev>0.030</stddev>
             </xacro:if>
             <xacro:unless value="$(arg sensor_noise)">

Commit message: chore: save baseline before slope-zero costmap experiment

File: src/lunar_rover_description/Rover_0/urdf/lunar_rover.urdf.xacro (robot description, xacro)
@@ -353,4 +353,239 @@
     <origin xyz="0 0 0" rpy="0 0 0"/>
   </joint>
+  <!--
+    5-DOF manipulator + parallel gripper (J1 yaw, J2/J3/J4 pitch, J5 jaw prismatic).
+    The base is mounted on the rover deck directly behind and above the Gemini335
+    depth camera (camera rear face x=0.1825, top z=0.0175). J2 sits directly above
+    J1. J2->J3, J3->J4, and J4->gripper working centre are all 0.115 m.
+    Folded zero pose: with every joint angle at zero the arm lies compactly on the
+    left side of the deck (x=0.13, y in [0, 0.108], z in [0.066, 0.181]). This
+    keeps it behind the Gemini335 lens and below the Mid-360 field of view. The
+    total arm mass is kept far below the rover mass. J1 = -pi/2 swings the folded
+    arm forward for manipulation.
+  -->
+  <xacro:property name="arm_base_x" value="0.13"/>
+  <xacro:property name="arm_base_z" value="0.056"/>
+  <xacro:property name="arm_j1_to_j2_z" value="0.09"/>
+  <xacro:property name="arm_upper_length" value="0.115"/>
+  <xacro:property name="arm_forearm_length" value="0.115"/>
+  <xacro:property name="arm_tool_length" value="0.115"/>
+  <!-- Zero-pose link directions in the link1/link2/link3 frames. -->
+  <xacro:property name="arm_upper_y" value="0.10782"/>
+  <xacro:property name="arm_upper_z" value="-0.04"/>
+  <xacro:property name="arm_forearm_y" value="-0.10782"/>
+  <xacro:property name="arm_forearm_z" value="-0.04"/>
+  <xacro:property name="arm_tool_z" value="0.115"/>
+  <xacro:property name="arm_link2_pitch" value="${atan2(-arm_upper_z, arm_upper_y)}"/>
+  <xacro:property name="arm_link3_pitch" value="${atan2(-arm_forearm_z, -arm_forearm_y)}"/>
+  <xacro:property name="arm_j1_lower" value="${-pi / 2.0}"/>
+  <xacro:property name="arm_j1_upper" value="${1.0}"/>
+  <xacro:property name="arm_pitch_lower" value="${-1.5}"/>
+  <xacro:property name="arm_pitch_upper" value="${1.5}"/>
+  <xacro:property name="arm_elbow_lower" value="${-2.0}"/>
+  <xacro:property name="arm_elbow_upper" value="${2.0}"/>
+  <xacro:property name="arm_gripper_stroke" value="0.045"/>
+  <xacro:property name="arm_finger_half_gap" value="0.012"/>
+  <xacro:property name="arm_finger_size" value="0.03 0.006 0.025"/>
+  <link name="arm_base_link">
+    <visual>
+      <geometry>
+        <box size="0.07 0.07 0.012"/>
+      </geometry>
+      <material name="suspension_dark"/>
+    </visual>
+    <collision>
+      <geometry>
+        <box size="0.07 0.07 0.012"/>
+      </geometry>
+    </collision>
+    <xacro:box_inertial mass="0.04" x="0.07" y="0.07" z="0.012"/>
+  </link>
+  <joint name="arm_base_joint" type="fixed">
+    <parent link="base_link"/>
+    <child link="arm_base_link"/>
+    <origin xyz="${arm_base_x} 0 ${arm_base_z}" rpy="0 0 0"/>
+  </joint>
+  <!-- J1: yaw axis. The shoulder riser keeps J2 directly above J1. -->
+  <link name="arm_link1">
+    <visual>
+      <origin xyz="0 0 ${arm_j1_to_j2_z / 2.0}" rpy="0 0 0"/>
+      <geometry>
+        <cylinder radius="0.03" length="${arm_j1_to_j2_z}"/>
+      </geometry>
+      <material name="suspension_dark"/>
+    </visual>
+    <collision>
+      <origin xyz="0 0 ${arm_j1_to_j2_z / 2.0}" rpy="0 0 0"/>
+      <geometry>
+        <cylinder radius="0.03" length="${arm_j1_to_j2_z}"/>
+      </geometry>
+    </collision>
+    <xacro:box_inertial mass="0.06" x="0.06" y="0.06" z="${arm_j1_to_j2_z}"/>
+  </link>
+  <joint name="arm_joint1" type="revolute">
+    <parent link="arm_base_link"/>
+    <child link="arm_link1"/>
+    <origin xyz="0 0 0" rpy="0 0 0"/>
+    <axis xyz="0 0 1"/>
+    <limit
+      lower="${arm_j1_lower}"
+      upper="${arm_j1_upper}"
+      effort="15.0"
+      velocity="1.5"/>
+    <dynamics damping="0.5" friction="0.1"/>
+  </joint>
+  <!-- J2: shoulder pitch, located at the top of the riser. -->
+  <link name="arm_link2">
+    <visual>
+      <origin xyz="0 ${arm_upper_y / 2.0} ${arm_upper_z / 2.0}" rpy="0 ${arm_link2_pitch} ${pi / 2.0}"/>
+      <geometry>
+        <box size="${arm_upper_length} 0.04 0.04"/>
+      </geometry>
+      <material name="chassis_white"/>
+    </visual>
+    <collision>
+      <origin xyz="0 ${arm_upper_y / 2.0} ${arm_upper_z / 2.0}" rpy="0 ${arm_link2_pitch} ${pi / 2.0}"/>
+      <geometry>
+        <box size="${arm_upper_length} 0.04 0.04"/>
+      </geometry>
+    </collision>
+    <xacro:box_inertial mass="0.08" x="${arm_upper_length}" y="0.04" z="0.04"/>
+  </link>
+  <joint name="arm_joint2" type="revolute">
+    <parent link="arm_link1"/>
+    <child link="arm_link2"/>
+    <origin xyz="0 0 ${arm_j1_to_j2_z}" rpy="0 0 0"/>
+    <axis xyz="0 1 0"/>
+    <limit
+      lower="${arm_pitch_lower}"
+      upper="${arm_pitch_upper}"
+      effort="15.0"
+      velocity="1.5"/>
+    <dynamics damping="0.5" friction="0.1"/>
+  </joint>
+  <!-- J3: elbow pitch. -->
+  <link name="arm_link3">
+    <visual>
+      <origin xyz="0 ${arm_forearm_y / 2.0} ${arm_forearm_z / 2.0}" rpy="0 ${arm_link3_pitch} ${-pi / 2.0}"/>
+      <geometry>
+        <box size="${arm_forearm_length} 0.04 0.04"/>
+      </geometry>
+      <material name="chassis_white"/>
+    </visual>
+    <collision>
+      <origin xyz="0 ${arm_forearm_y / 2.0} ${arm_forearm_z / 2.0}" rpy="0 ${arm_link3_pitch} ${-pi / 2.0}"/>
+      <geometry>
+        <box size="${arm_forearm_length} 0.04 0.04"/>
+      </geometry>
+    </collision>
+    <xacro:box_inertial mass="0.06" x="${arm_forearm_length}" y="0.04" z="0.04"/>
+  </link>
+  <joint name="arm_joint3" type="revolute">
+    <parent link="arm_link2"/>
+    <child link="arm_link3"/>
+    <origin xyz="0 ${arm_upper_y} ${arm_upper_z}" rpy="0 0 0"/>
+    <axis xyz="0 1 0"/>
+    <limit
+      lower="${arm_elbow_lower}"
+      upper="${arm_elbow_upper}"
+      effort="12.0"
+      velocity="1.8"/>
+    <dynamics damping="0.4" friction="0.08"/>
+  </joint>
+  <!-- J4: wrist pitch. The palm carries the fixed gripper finger and J5's jaw. -->
+  <link name="arm_link4">
+    <visual>
+      <origin xyz="0 0 ${arm_tool_z / 2.0}" rpy="0 0 0"/>
+      <geometry>
+        <box size="0.04 0.04 ${arm_tool_length}"/>
+      </geometry>
+      <material name="chassis_white"/>
+    </visual>
+    <visual>
+      <origin xyz="0 ${-arm_finger_half_gap} ${arm_tool_z}" rpy="0 0 0"/>
+      <geometry>
+        <box size="${arm_finger_size}"/>
+      </geometry>
+      <material name="camera_black"/>
+    </visual>
+    <collision>
+      <origin xyz="0 0 ${arm_tool_z / 2.0}" rpy="0 0 0"/>
+      <geometry>
+        <box size="0.04 0.04 ${arm_tool_length}"/>
+      </geometry>
+    </collision>
+    <collision>
+      <origin xyz="0 ${-arm_finger_half_gap} ${arm_tool_z}" rpy="0 0 0"/>
+      <geometry>
+        <box size="${arm_finger_size}"/>
+      </geometry>
+    </collision>
+    <xacro:box_inertial mass="0.06" x="0.04" y="0.04" z="${arm_tool_length}"/>
+  </link>
+  <joint name="arm_joint4" type="revolute">
+    <parent link="arm_link3"/>
+    <child link="arm_link4"/>
+    <origin xyz="0 ${arm_forearm_y} ${arm_forearm_z}" rpy="0 0 0"/>
+    <axis xyz="0 1 0"/>
+    <limit
+      lower="${arm_pitch_lower}"
+      upper="${arm_pitch_upper}"
+      effort="10.0"
+      velocity="2.0"/>
+    <dynamics damping="0.4" friction="0.08"/>
+  </joint>
+  <!-- J5: prismatic gripper jaw. The fixed finger is part of arm_link4; the
+       moving finger travels along +y so the mid-point is the working centre. -->
+  <link name="arm_link5">
+    <visual>
+      <origin xyz="0 ${arm_finger_half_gap} 0" rpy="0 0 0"/>
+      <geometry>
+        <box size="${arm_finger_size}"/>
+      </geometry>
+      <material name="camera_black"/>
+    </visual>
+    <collision>
+      <origin xyz="0 ${arm_finger_half_gap} 0" rpy="0 0 0"/>
+      <geometry>
+        <box size="${arm_finger_size}"/>
+      </geometry>
+    </collision>
+    <xacro:box_inertial mass="0.005" x="0.03" y="0.006" z="0.025"/>
+  </link>
+  <joint name="arm_joint5" type="prismatic">
+    <parent link="arm_link4"/>
+    <child link="arm_link5"/>
+    <origin xyz="0 0 ${arm_tool_z}" rpy="0 0 0"/>
+    <axis xyz="0 1 0"/>
+    <limit
+      lower="0.0"
+      upper="${arm_gripper_stroke}"
+      effort="8.0"
+      velocity="0.12"/>
+    <dynamics damping="0.6" friction="0.15"/>
+  </joint>
+  <!--
+    Disable collisions between the arm links and every other link of the same
+    rover model. URDF-to-SDF conversion defaults <self_collide> to false, so
+    adjacent boxes/cylinders at J2/J3/J4 and the folded zero pose would push
+    against each other and cause contact jitter under position control. The
+    fingers still collide with external objects (rocks, sample blocks) because
+    those are separate Gazebo models.
+  -->
+  <gazebo reference="arm_link1">
+    <selfCollide>true</selfCollide>
+  </gazebo>
+  <gazebo reference="arm_link2">
+    <selfCollide>true</selfCollide>
+  </gazebo>
+  <gazebo reference="arm_link3">
+    <selfCollide>true</selfCollide>
+  </gazebo>
+  <gazebo reference="arm_link4">
+    <selfCollide>true</selfCollide>
+  </gazebo>
+  <gazebo reference="arm_link5">
+    <selfCollide>true</selfCollide>
+  </gazebo>
   <ros2_control name="LunarRoverSystem" type="system">
     <hardware>
@@ -458,4 +693,44 @@
     </joint>
     <joint name="right_bogie_joint">
+      <state_interface name="position"/>
+      <state_interface name="velocity"/>
+    </joint>
+    <joint name="arm_joint1">
+      <command_interface name="position">
+        <param name="min">${arm_j1_lower}</param>
+        <param name="max">${arm_j1_upper}</param>
+      </command_interface>
+      <state_interface name="position"/>
+      <state_interface name="velocity"/>
+    </joint>
+    <joint name="arm_joint2">
+      <command_interface name="position">
+        <param name="min">${arm_pitch_lower}</param>
+        <param name="max">${arm_pitch_upper}</param>
+      </command_interface>
+      <state_interface name="position"/>
+      <state_interface name="velocity"/>
+    </joint>
+    <joint name="arm_joint3">
+      <command_interface name="position">
+        <param name="min">${arm_elbow_lower}</param>
+        <param name="max">${arm_elbow_upper}</param>
+      </command_interface>
+      <state_interface name="position"/>
+      <state_interface name="velocity"/>
+    </joint>
+    <joint name="arm_joint4">
+      <command_interface name="position">
+        <param name="min">${arm_pitch_lower}</param>
+        <param name="max">${arm_pitch_upper}</param>
+      </command_interface>
+      <state_interface name="position"/>
+      <state_interface name="velocity"/>
+    </joint>
+    <joint name="arm_joint5">
+      <command_interface name="position">
+        <param name="min">0.0</param>
+        <param name="max">${arm_gripper_stroke}</param>
+      </command_interface>
       <state_interface name="position"/>
       <state_interface name="velocity"/>

Commit message: feat: add real rover visual grasp pipeline

File: src/lunar_rover_description/Rover_0/urdf/lunar_rover.urdf.xacro (robot description, xacro)
@@ -7,4 +7,6 @@
     name="ros2_control_hardware_plugin"
     default="gz_ros2_control/GazeboSimSystem"/>
+  <xacro:arg name="arm_camera_xyz" default="0.04 0 0.065"/>
+  <xacro:arg name="arm_camera_rpy" default="0 -1.57079632679 0"/>
   <!-- Compact rover envelope: 0.54 m long x 0.40 m wide including wheels. -->
   <xacro:property name="track" value="0.345"/>
@@ -294,5 +296,5 @@
     <parent link="sensor_mast_link"/>
     <child link="mid360_link"/>
-    <origin xyz="0 0 0.155" rpy="0 ${35.0 * pi / 180.0} 0"/>
+    <origin xyz="0 0 0.155" rpy="0 ${45.0 * pi / 180.0} 0"/>
   </joint>
   <link name="livox_frame"/>
@@ -323,8 +325,13 @@
     <xacro:box_inertial mass="0.097" x="0.030" y="0.090" z="0.025"/>
   </link>
+  <!--
+    Legacy coarse camera mount retained for the old Rover_0 simulation / MoveIt
+    path only. As of 2026-08-30, do not treat this mount as the real-arm
+    hand-eye truth; use the temporary hand-eye TF chain instead.
+  -->
   <joint name="gemini335_joint" type="fixed">
-    <parent link="base_link"/>
+    <parent link="arm_link4"/>
     <child link="gemini335_link"/>
-    <origin xyz="0.1975 0 0.005" rpy="0 0 0"/>
+    <origin xyz="$(arg arm_camera_xyz)" rpy="$(arg arm_camera_rpy)"/>
   </joint>
   <link name="gemini335_color_optical_frame"/>
@@ -353,35 +360,17 @@
     <origin xyz="0 0 0" rpy="0 0 0"/>
   </joint>
-  <!--
-    5-DOF manipulator + parallel gripper (J1 yaw, J2/J3/J4 pitch, J5 jaw prismatic).
-    The base is mounted on the rover deck directly behind and above the Gemini335
-    depth camera (camera rear face x=0.1825, top z=0.0175). J2 sits directly above
-    J1. J2->J3, J3->J4, and J4->gripper working centre are all 0.115 m.
-    Folded zero pose: with every joint angle at zero the arm lies compactly on the
-    left side of the deck (x=0.13, y in [0, 0.108], z in [0.066, 0.181]). This
-    keeps it behind the Gemini335 lens and below the Mid-360 field of view. The
-    total arm mass is kept far below the rover mass. J1 = -pi/2 swings the folded
-    arm forward for manipulation.
-  -->
+  <!-- Real arm geometry. ROS zero equals servo Home: 90/180/135/135 degrees. -->
   <xacro:property name="arm_base_x" value="0.13"/>
   <xacro:property name="arm_base_z" value="0.056"/>
-  <xacro:property name="arm_j1_to_j2_z" value="0.09"/>
-  <xacro:property name="arm_upper_length" value="0.115"/>
-  <xacro:property name="arm_forearm_length" value="0.115"/>
-  <xacro:property name="arm_tool_length" value="0.115"/>
-  <!-- Zero-pose link directions in the link1/link2/link3 frames. -->
-  <xacro:property name="arm_upper_y" value="0.10782"/>
-  <xacro:property name="arm_upper_z" value="-0.04"/>
-  <xacro:property name="arm_forearm_y" value="-0.10782"/>
-  <xacro:property name="arm_forearm_z" value="-0.04"/>
-  <xacro:property name="arm_tool_z" value="0.115"/>
-  <xacro:property name="arm_link2_pitch" value="${atan2(-arm_upper_z, arm_upper_y)}"/>
-  <xacro:property name="arm_link3_pitch" value="${atan2(-arm_forearm_z, -arm_forearm_y)}"/>
+  <xacro:property name="arm_j1_to_j2_z" value="0.07545"/>
+  <xacro:property name="arm_upper_length" value="0.11391"/>
+  <xacro:property name="arm_forearm_length" value="0.11000"/>
+  <xacro:property name="arm_tool_length" value="0.15601"/>
   <xacro:property name="arm_j1_lower" value="${-pi / 2.0}"/>
-  <xacro:property name="arm_j1_upper" value="${1.0}"/>
+  <xacro:property name="arm_j1_upper" value="${pi}"/>
   <xacro:property name="arm_pitch_lower" value="${-1.5}"/>
-  <xacro:property name="arm_pitch_upper" value="${1.5}"/>
-  <xacro:property name="arm_elbow_lower" value="${-2.0}"/>
-  <xacro:property name="arm_elbow_upper" value="${2.0}"/>
+  <xacro:property name="arm_pitch_upper" value="${pi}"/>
+  <xacro:property name="arm_elbow_lower" value="${-3.0 * pi / 4.0}"/>
+  <xacro:property name="arm_elbow_upper" value="${3.0 * pi / 4.0}"/>
   <xacro:property name="arm_gripper_stroke" value="0.045"/>
   <xacro:property name="arm_finger_half_gap" value="0.012"/>
@@ -438,17 +427,17 @@
   <link name="arm_link2">
     <visual>
-      <origin xyz="0 ${arm_upper_y / 2.0} ${arm_upper_z / 2.0}" rpy="0 ${arm_link2_pitch} ${pi / 2.0}"/>
-      <geometry>
-        <box size="${arm_upper_length} 0.04 0.04"/>
+      <origin xyz="0 0 ${arm_upper_length / 2.0}" rpy="0 0 0"/>
+      <geometry>
+        <box size="0.04 0.04 ${arm_upper_length}"/>
       </geometry>
       <material name="chassis_white"/>
     </visual>
     <collision>
-      <origin xyz="0 ${arm_upper_y / 2.0} ${arm_upper_z / 2.0}" rpy="0 ${arm_link2_pitch} ${pi / 2.0}"/>
-      <geometry>
-        <box size="${arm_upper_length} 0.04 0.04"/>
-      </geometry>
-    </collision>
-    <xacro:box_inertial mass="0.08" x="${arm_upper_length}" y="0.04" z="0.04"/>
+      <origin xyz="0 0 ${arm_upper_length / 2.0}" rpy="0 0 0"/>
+      <geometry>
+        <box size="0.04 0.04 ${arm_upper_length}"/>
+      </geometry>
+    </collision>
+    <xacro:box_inertial mass="0.08" x="0.04" y="0.04" z="${arm_upper_length}"/>
   </link>
   <joint name="arm_joint2" type="revolute">
@@ -467,22 +456,22 @@
   <link name="arm_link3">
     <visual>
-      <origin xyz="0 ${arm_forearm_y / 2.0} ${arm_forearm_z / 2.0}" rpy="0 ${arm_link3_pitch} ${-pi / 2.0}"/>
-      <geometry>
-        <box size="${arm_forearm_length} 0.04 0.04"/>
+      <origin xyz="0 0 ${arm_forearm_length / 2.0}" rpy="0 0 0"/>
+      <geometry>
+        <box size="0.04 0.04 ${arm_forearm_length}"/>
       </geometry>
       <material name="chassis_white"/>
     </visual>
     <collision>
-      <origin xyz="0 ${arm_forearm_y / 2.0} ${arm_forearm_z / 2.0}" rpy="0 ${arm_link3_pitch} ${-pi / 2.0}"/>
-      <geometry>
-        <box size="${arm_forearm_length} 0.04 0.04"/>
-      </geometry>
-    </collision>
-    <xacro:box_inertial mass="0.06" x="${arm_forearm_length}" y="0.04" z="0.04"/>
+      <origin xyz="0 0 ${arm_forearm_length / 2.0}" rpy="0 0 0"/>
+      <geometry>
+        <box size="0.04 0.04 ${arm_forearm_length}"/>
+      </geometry>
+    </collision>
+    <xacro:box_inertial mass="0.06" x="0.04" y="0.04" z="${arm_forearm_length}"/>
   </link>
   <joint name="arm_joint3" type="revolute">
     <parent link="arm_link2"/>
     <child link="arm_link3"/>
-    <origin xyz="0 ${arm_upper_y} ${arm_upper_z}" rpy="0 0 0"/>
+    <origin xyz="0 0 ${arm_upper_length}" rpy="0 0 0"/>
     <axis xyz="0 1 0"/>
     <limit
@@ -496,5 +485,5 @@
   <link name="arm_link4">
     <visual>
-      <origin xyz="0 0 ${arm_tool_z / 2.0}" rpy="0 0 0"/>
+      <origin xyz="0 0 ${arm_tool_length / 2.0}" rpy="0 0 0"/>
       <geometry>
         <box size="0.04 0.04 ${arm_tool_length}"/>
@@ -503,5 +492,5 @@
     </visual>
     <visual>
-      <origin xyz="0 ${-arm_finger_half_gap} ${arm_tool_z}" rpy="0 0 0"/>
+      <origin xyz="0 ${-arm_finger_half_gap} ${arm_tool_length}" rpy="0 0 0"/>
       <geometry>
         <box size="${arm_finger_size}"/>
@@ -510,5 +499,5 @@
     </visual>
     <collision>
-      <origin xyz="0 0 ${arm_tool_z / 2.0}" rpy="0 0 0"/>
+      <origin xyz="0 0 ${arm_tool_length / 2.0}" rpy="0 0 0"/>
       <geometry>
         <box size="0.04 0.04 ${arm_tool_length}"/>
@@ -516,5 +505,5 @@
     </collision>
     <collision>
-      <origin xyz="0 ${-arm_finger_half_gap} ${arm_tool_z}" rpy="0 0 0"/>
+      <origin xyz="0 ${-arm_finger_half_gap} ${arm_tool_length}" rpy="0 0 0"/>
       <geometry>
         <box size="${arm_finger_size}"/>
@@ -526,5 +515,5 @@
     <parent link="arm_link3"/>
     <child link="arm_link4"/>
-    <origin xyz="0 ${arm_forearm_y} ${arm_forearm_z}" rpy="0 0 0"/>
+    <origin xyz="0 0 ${arm_forearm_length}" rpy="0 0 0"/>
     <axis xyz="0 1 0"/>
     <limit
@@ -556,5 +545,5 @@
     <parent link="arm_link4"/>
     <child link="arm_link5"/>
-    <origin xyz="0 0 ${arm_tool_z}" rpy="0 0 0"/>
+    <origin xyz="0 0 ${arm_tool_length}" rpy="0 0 0"/>
     <axis xyz="0 1 0"/>
     <limit
